Commit message: updated urdf with correct values

File: mbot_description/urdf/mbot_classic.urdf.xacro (robot description, xacro)
@@ -8,33 +8,10 @@
       <color rgba="0.0 0.0 0.8 1.0"/>
   </material>
-  <!-- Specify some standard inertial calculations https://en.wikipedia.org/wiki/List_of_moments_of_inertia -->
-  <!-- These make use of xacro's mathematical functionality -->
-  <xacro:macro name="inertial_sphere" params="mass radius *origin">
-      <inertial>
-          <xacro:insert_block name="origin"/>
-          <mass value="${mass}" />
-          <inertia ixx="${(2/5) * mass * (radius*radius)}" ixy="0.0" ixz="0.0"
-                  iyy="${(2/5) * mass * (radius*radius)}" iyz="0.0"
-                  izz="${(2/5) * mass * (radius*radius)}" />
-      </inertial>
-  </xacro:macro>
-  <xacro:macro name="inertial_box" params="mass x y z *origin">
-      <inertial>
-          <xacro:insert_block name="origin"/>
-          <mass value="${mass}" />
-          <inertia ixx="${(1/12) * mass * (y*y+z*z)}" ixy="0.0" ixz="0.0"
-                  iyy="${(1/12) * mass * (x*x+z*z)}" iyz="0.0"
-                  izz="${(1/12) * mass * (x*x+y*y)}" />
-      </inertial>
-  </xacro:macro>
-  <xacro:macro name="inertial_cylinder" params="mass length radius *origin">
-      <inertial>
-          <xacro:insert_block name="origin"/>
-          <mass value="${mass}" />
-          <inertia ixx="${(1/12) * mass * (3*radius*radius + length*length)}" ixy="0.0" ixz="0.0"
-                  iyy="${(1/12) * mass * (3*radius*radius + length*length)}" iyz="0.0"
-                  izz="${(1/2) * mass * (radius*radius)}" />
-      </inertial>
-  </xacro:macro>
+  <material name="yellow">
+      <color rgba="0.8 0.8 0.0 1.0"/>
+  </material>
+  <material name="green">
+      <color rgba="0.0 0.8 0.0 1.0"/>
+  </material>
 <!-- ===================== MAIN BODY =========================== -->
   <link name="base_footprint"/>
@@ -43,5 +20,5 @@
     <parent link="base_footprint"/>
     <child link="base_link"/>
-    <origin xyz="0 0 0.041" rpy="0 0 0"/>
+    <origin xyz="0 0 0.042" rpy="0 0 0"/>
   </joint>
   <!-- CHASSIS -->
@@ -49,7 +26,7 @@
     <visual>
       <geometry>
-        <box size="0.18 0.13 0.095"/>
+        <box size="0.17 0.13 0.005"/>
       </geometry>
-      <origin rpy="0 0 0" xyz="-0.045 0 0.0275"/>
+      <origin rpy="0 0 0" xyz="-0.038 0 -0.0115"/>
       <material name="blue"/>
     </visual>
@@ -58,15 +35,74 @@
         <box size="0.18 0.13 0.095"/>
       </geometry>
-      <origin rpy="0 0 0" xyz="-0.045 0 0.0275"/>
+      <origin rpy="0 0 0" xyz="-0.038 0 -0.0115"/>
     </collision>
-    <xacro:inertial_box mass="0.3" x="0.18" y="0.13" z="0.095">
-      <origin xyz="0 0 0.0275" rpy="0 0 0"/>
-    </xacro:inertial_box>
   </link>
+  <!-- MIDDLE AND TOP LAYERS -->
+  <link name="middle_link">
+    <visual>
+      <geometry>
+        <box size="0.144 0.13 0.005"/>
+      </geometry>
+      <origin rpy="0 0 0" xyz="-0.025 0 0"/>
+      <material name="yellow"/>
+    </visual>
+    <collision>
+      <geometry>
+        <box size="0.144 0.13 0.005"/>
+      </geometry>
+      <origin rpy="0 0 0" xyz="-0.025 0 0"/>
+    </collision>
+  </link>
+  <link name="top_link">
+    <visual>
+      <geometry>
+        <box size="0.144 0.13 0.005"/>
+      </geometry>
+      <origin rpy="0 0 0" xyz="-0.025 0 0"/>
+      <material name="blue"/>
+    </visual>
+    <collision>
+      <geometry>
+        <box size="0.144 0.13 0.005"/>
+      </geometry>
+      <origin rpy="0 0 0" xyz="-0.025 0 0"/>
+    </collision>
+  </link>
+  <joint name="middle_joint" type="fixed">
+    <parent link="base_link"/>
+    <child link="middle_link"/>
+    <origin xyz="0 0 0.02936" rpy="0 0 0"/>
+  </joint>
+  <joint name="top_joint" type="fixed">
+    <parent link="middle_link"/>
+    <child link="top_link"/>
+    <origin xyz="0 0 0.067" rpy="0 0 0"/>
+  </joint>
+  <!-- CAMERA on middle layer -->
+  <link name="camera_link">
+    <visual>
+      <geometry>
+        <box size="0.005 0.05 0.05"/>
+      </geometry>
+      <origin rpy="0 0 0" xyz="0 0 0"/>
+      <material name="green"/>
+    </visual>
+    <collision>
+      <geometry>
+        <box size="0.005 0.05 0.05"/>
+      </geometry>
+      <origin rpy="0 0 0" xyz="0 0 0"/>
+    </collision>
+  </link>
+  <joint name="camera_joint" type="fixed">
+    <parent link="base_link"/>
+    <child link="camera_link"/>
+    <origin xyz="0.05751 0 0.02936" rpy="0 0 0"/>
+  </joint>
   <!-- WHEELS -->
   <link name="left_wheel_link">
     <visual>
       <geometry>
-        <cylinder radius="0.041" length="0.02"/>
+        <cylinder radius="0.042" length="0.024"/>
       </geometry>
       <origin rpy="0 0 0" xyz="0 0 0"/>
@@ -75,16 +111,13 @@
     <collision>
       <geometry>
-        <cylinder radius="0.041" length="0.02"/>
+        <cylinder radius="0.042" length="0.024"/>
       </geometry>
       <origin rpy="0 0 0" xyz="0 0 0"/>
     </collision>
-    <xacro:inertial_cylinder mass="0.1" length="0.02" radius="0.041">
-      <origin xyz="0 0 0" rpy="0 0 0"/>
-    </xacro:inertial_cylinder>
   </link>
   <link name="right_wheel_link">
     <visual>
       <geometry>
-        <cylinder radius="0.041" length="0.02"/>
+        <cylinder radius="0.042" length="0.024"/>
       </geometry>
       <origin rpy="0 0 0" xyz="0 0 0"/>
@@ -93,11 +126,8 @@
     <collision>
       <geometry>
-        <cylinder radius="0.041" length="0.02"/>
+        <cylinder radius="0.042" length="0.024"/>
       </geometry>
       <origin rpy="0 0 0" xyz="0 0 0"/>
     </collision>
-    <xacro:inertial_cylinder mass="0.1" length="0.02" radius="0.041">
-      <origin xyz="0 0 0" rpy="0 0 0"/>
-    </xacro:inertial_cylinder>
   </link>
   <joint name="left_wheel_joint" type="continuous">
@@ -106,6 +136,4 @@
     <origin xyz="0 0.085 0" rpy="-1.5708 0 0"/>
     <axis xyz="0 0 1"/>
-    <limit effort="5000" velocity="10"/>
-    <dynamics damping="1.0" friction="1.0"/>
   </joint>
   <joint name="right_wheel_joint" type="continuous">
@@ -114,35 +142,10 @@
     <origin xyz="0 -0.085 0" rpy="1.5708 0 0"/>
     <axis xyz="0 0 -1"/>
-    <limit effort="5000" velocity="10"/>
-    <dynamics damping="1.0" friction="1.0"/>
   </joint>
-  <!-- CASTER (Support ball that can roll freely) -->
-  <!-- Set to fixed joint but also set friction to 0 -->
-  <joint name="caster_wheel_joint" type="fixed">
-    <parent link="base_link"/>
-    <child link="caster_wheel_link"/>
-    <origin xyz="-0.09 0 0"/>
-  </joint>
-  <link name="caster_wheel_link">
-    <visual>
-      <geometry>
-        <sphere radius="0.041"/>
-      </geometry>
-      <material name="black"/>
-    </visual>
-    <collision>
-      <geometry>
-        <sphere radius="0.041"/>
-      </geometry>
-    </collision>
-    <xacro:inertial_sphere mass="0.1" radius="0.041">
-      <origin xyz="0 0 0" rpy="0 0 0"/>
-    </xacro:inertial_sphere>
-  </link>
   <!-- RPLidar A1 (Directly above base_link) -->
   <link name="lidar_link">
     <visual>
       <geometry>
-        <cylinder radius="0.049" length="0.041"/>
+        <cylinder radius="0.0336" length="0.022"/>
       </geometry>
       <origin rpy="0 0 0" xyz="0 0 0"/>
@@ -151,16 +154,13 @@
     <collision>
       <geometry>
-        <cylinder radius="0.049" length="0.041"/>
+        <cylinder radius="0.0336" length="0.022"/>
       </geometry>
       <origin rpy="0 0 0" xyz="0 0 0"/>
     </collision>
-    <xacro:inertial_cylinder mass="0.1" length="0.041" radius="0.049">
-      <origin xyz="0 0 0" rpy="0 0 0"/>
-    </xacro:inertial_cylinder>
   </link>
   <joint name="lidar_joint" type="fixed">
     <parent link="base_link"/>
     <child link="lidar_link"/>
-    <origin xyz="0 0 0.1" rpy="0 0 3.14"/>
+    <origin xyz="0 0 0.14179" rpy="0 0 3.14"/>
   </joint>
 </robot>

Commit message: added meshes

File: mbot_description/urdf/mbot_classic.urdf.xacro (robot description, xacro)
@@ -6,5 +6,5 @@
   </material>
   <material name="blue">
-      <color rgba="0.0 0.0 0.8 1.0"/>
+      <color rgba="0.07 0.08 0.7 1.0"/>
   </material>
   <material name="yellow">
@@ -27,4 +27,5 @@
       <geometry>
         <box size="0.17 0.13 0.005"/>
+        <!-- <mesh filename="package://mbot_description/meshes/base.dae" scale="0.001 0.001 0.001"/> -->
       </geometry>
       <origin rpy="0 0 0" xyz="-0.038 0 -0.0115"/>
@@ -57,7 +58,8 @@
     <visual>
       <geometry>
-        <box size="0.144 0.13 0.005"/>
+        <!-- <box size="0.144 0.13 0.005"/> -->
+        <mesh filename="package://mbot_description/meshes/top.stl" scale="0.001 0.001 0.001"/>
       </geometry>
-      <origin rpy="0 0 0" xyz="-0.025 0 0"/>
+      <origin rpy="0 0 3.14" xyz="0 0 0"/>
       <material name="blue"/>
     </visual>
@@ -83,8 +85,8 @@
     <visual>
       <geometry>
-        <box size="0.005 0.05 0.05"/>
+        <mesh filename="package://mbot_description/meshes/camera-set.dae" scale="0.001 0.001 0.001"/>
       </geometry>
       <origin rpy="0 0 0" xyz="0 0 0"/>
-      <material name="green"/>
+      <!-- <material name="green"/> -->
     </visual>
     <collision>
@@ -104,5 +106,5 @@
     <visual>
       <geometry>
-        <cylinder radius="0.042" length="0.024"/>
+        <mesh filename="package://mbot_description/meshes/wheel_l.stl" scale="0.001 0.001 0.001"/>
       </geometry>
       <origin rpy="0 0 0" xyz="0 0 0"/>
@@ -115,9 +117,9 @@
       <origin rpy="0 0 0" xyz="0 0 0"/>
     </collision>
-  </link>
+      </link>
   <link name="right_wheel_link">
     <visual>
       <geometry>
-        <cylinder radius="0.042" length="0.024"/>
+        <mesh filename="package://mbot_description/meshes/wheel_r.stl" scale="0.001 0.001 0.001"/>
       </geometry>
       <origin rpy="0 0 0" xyz="0 0 0"/>
@@ -147,7 +149,8 @@
     <visual>
       <geometry>
-        <cylinder radius="0.0336" length="0.022"/>
+        <!-- <cylinder radius="0.0336" length="0.022"/> -->
+        <mesh filename="package://mbot_description/meshes/lidar.dae" scale="0.001 0.001 0.001"/>
       </geometry>
-      <origin rpy="0 0 0" xyz="0 0 0"/>
+      <origin rpy="0 0 0" xyz="0 0 -0.04375"/>
       <material name="black"/>
     </visual>

Commit message: finalized urdf model

File: mbot_description/urdf/mbot_classic.urdf.xacro (robot description, xacro)
@@ -1,17 +1,7 @@
 <?xml version="1.0"?>
 <robot xmlns:xacro="http://www.ros.org/wiki/xacro" name="mbot">
-  <!-- Init colour -->
-  <material name="black">
-      <color rgba="0.2 0.2 0.2 1.0"/>
-  </material>
-  <material name="blue">
-      <color rgba="0.07 0.08 0.7 1.0"/>
-  </material>
-  <material name="yellow">
-      <color rgba="0.8 0.8 0.0 1.0"/>
-  </material>
-  <material name="green">
-      <color rgba="0.0 0.8 0.0 1.0"/>
-  </material>
+<material name="black">
+    <color rgba="0.2 0.2 0.2 1.0"/>
+</material>
 <!-- ===================== MAIN BODY =========================== -->
   <link name="base_footprint"/>
@@ -26,9 +16,7 @@
     <visual>
       <geometry>
-        <box size="0.17 0.13 0.005"/>
-        <!-- <mesh filename="package://mbot_description/meshes/base.dae" scale="0.001 0.001 0.001"/> -->
+        <mesh filename="package://mbot_description/meshes/mbot-classic-simplied.dae"/>
       </geometry>
-      <origin rpy="0 0 0" xyz="-0.038 0 -0.0115"/>
-      <material name="blue"/>
+      <origin rpy="0 0 0" xyz="-0.04 -0.115 0.005"/>
     </visual>
     <collision>
@@ -36,65 +24,9 @@
         <box size="0.18 0.13 0.095"/>
       </geometry>
-      <origin rpy="0 0 0" xyz="-0.038 0 -0.0115"/>
+      <origin rpy="0 0 0" xyz="-0.04 -0.115 0.005"/>
     </collision>
   </link>
-  <!-- MIDDLE AND TOP LAYERS -->
-  <link name="middle_link">
-    <visual>
-      <geometry>
-        <box size="0.144 0.13 0.005"/>
-      </geometry>
-      <origin rpy="0 0 0" xyz="-0.025 0 0"/>
-      <material name="yellow"/>
-    </visual>
-    <collision>
-      <geometry>
-        <box size="0.144 0.13 0.005"/>
-      </geometry>
-      <origin rpy="0 0 0" xyz="-0.025 0 0"/>
-    </collision>
-  </link>
-  <link name="top_link">
-    <visual>
-      <geometry>
-        <!-- <box size="0.144 0.13 0.005"/> -->
-        <mesh filename="package://mbot_description/meshes/top.stl" scale="0.001 0.001 0.001"/>
-      </geometry>
-      <origin rpy="0 0 3.14" xyz="0 0 0"/>
-      <material name="blue"/>
-    </visual>
-    <collision>
-      <geometry>
-        <box size="0.144 0.13 0.005"/>
-      </geometry>
-      <origin rpy="0 0 0" xyz="-0.025 0 0"/>
-    </collision>
-  </link>
-  <joint name="middle_joint" type="fixed">
-    <parent link="base_link"/>
-    <child link="middle_link"/>
-    <origin xyz="0 0 0.02936" rpy="0 0 0"/>
-  </joint>
-  <joint name="top_joint" type="fixed">
-    <parent link="middle_link"/>
-    <child link="top_link"/>
-    <origin xyz="0 0 0.067" rpy="0 0 0"/>
-  </joint>
-  <!-- CAMERA on middle layer -->
-  <link name="camera_link">
-    <visual>
-      <geometry>
-        <mesh filename="package://mbot_description/meshes/camera-set.dae" scale="0.001 0.001 0.001"/>
-      </geometry>
-      <origin rpy="0 0 0" xyz="0 0 0"/>
-      <!-- <material name="green"/> -->
-    </visual>
-    <collision>
-      <geometry>
-        <box size="0.005 0.05 0.05"/>
-      </geometry>
-      <origin rpy="0 0 0" xyz="0 0 0"/>
-    </collision>
-  </link>
+  <!-- CAMERA -->
+  <link name="camera_link"/>
   <joint name="camera_joint" type="fixed">
     <parent link="base_link"/>
@@ -108,5 +40,5 @@
         <mesh filename="package://mbot_description/meshes/wheel_l.stl" scale="0.001 0.001 0.001"/>
       </geometry>
-      <origin rpy="0 0 0" xyz="0 0 0"/>
+      <origin rpy="0 0 0" xyz="0 0 0.0115"/>
       <material name="black"/>
     </visual>
@@ -115,5 +47,5 @@
         <cylinder radius="0.042" length="0.024"/>
       </geometry>
-      <origin rpy="0 0 0" xyz="0 0 0"/>
+      <origin rpy="0 0 0" xyz="0 0 0.0115"/>
     </collision>
       </link>
@@ -123,5 +55,5 @@
         <mesh filename="package://mbot_description/meshes/wheel_r.stl" scale="0.001 0.001 0.001"/>
       </geometry>
-      <origin rpy="0 0 0" xyz="0 0 0"/>
+      <origin rpy="0 0 0" xyz="0 0 0.0115"/>
       <material name="black"/>
     </visual>
@@ -130,5 +62,5 @@
         <cylinder radius="0.042" length="0.024"/>
       </geometry>
-      <origin rpy="0 0 0" xyz="0 0 0"/>
+      <origin rpy="0 0 0" xyz="0 0 0.0115"/>
     </collision>
   </link>
@@ -146,20 +78,5 @@
   </joint>
   <!-- RPLidar A1 (Directly above base_link) -->
-  <link name="lidar_link">
-    <visual>
-      <geometry>
-        <!-- <cylinder radius="0.0336" length="0.022"/> -->
-        <mesh filename="package://mbot_description/meshes/lidar.dae" scale="0.001 0.001 0.001"/>
-      </geometry>
-      <origin rpy="0 0 0" xyz="0 0 -0.04375"/>
-      <material name="black"/>
-    </visual>
-    <collision>
-      <geometry>
-        <cylinder radius="0.0336" length="0.022"/>
-      </geometry>
-      <origin rpy="0 0 0" xyz="0 0 0"/>
-    </collision>
-  </link>
+  <link name="lidar_link"/>
   <joint name="lidar_joint" type="fixed">
     <parent link="base_link"/>

Commit message: Finalized URDF + Added README (#5)
* clean up gazebo legacy code

* updated urdf with correct values

* added meshes

* finalized urdf model

* updated the readme file

File: mbot_description/urdf/mbot_classic.urdf.xacro (robot description, xacro)
@@ -1,42 +1,7 @@
 <?xml version="1.0"?>
 <robot xmlns:xacro="http://www.ros.org/wiki/xacro" name="mbot">
-  <!-- Include Gazebo control -->
-  <xacro:include filename="$(find mbot_description)/urdf/mbot.gazebo"/>
-  <!-- Init colour -->
-  <material name="black">
-      <color rgba="0.2 0.2 0.2 1.0"/>
-  </material>
-  <material name="blue">
-      <color rgba="0.0 0.0 0.8 1.0"/>
-  </material>
-  <!-- Specify some standard inertial calculations https://en.wikipedia.org/wiki/List_of_moments_of_inertia -->
-  <!-- These make use of xacro's mathematical functionality -->
-  <xacro:macro name="inertial_sphere" params="mass radius *origin">
-      <inertial>
-          <xacro:insert_block name="origin"/>
-          <mass value="${mass}" />
-          <inertia ixx="${(2/5) * mass * (radius*radius)}" ixy="0.0" ixz="0.0"
-                  iyy="${(2/5) * mass * (radius*radius)}" iyz="0.0"
-                  izz="${(2/5) * mass * (radius*radius)}" />
-      </inertial>
-  </xacro:macro>
-  <xacro:macro name="inertial_box" params="mass x y z *origin">
-      <inertial>
-          <xacro:insert_block name="origin"/>
-          <mass value="${mass}" />
-          <inertia ixx="${(1/12) * mass * (y*y+z*z)}" ixy="0.0" ixz="0.0"
-                  iyy="${(1/12) * mass * (x*x+z*z)}" iyz="0.0"
-                  izz="${(1/12) * mass * (x*x+y*y)}" />
-      </inertial>
-  </xacro:macro>
-  <xacro:macro name="inertial_cylinder" params="mass length radius *origin">
-      <inertial>
-          <xacro:insert_block name="origin"/>
-          <mass value="${mass}" />
-          <inertia ixx="${(1/12) * mass * (3*radius*radius + length*length)}" ixy="0.0" ixz="0.0"
-                  iyy="${(1/12) * mass * (3*radius*radius + length*length)}" iyz="0.0"
-                  izz="${(1/2) * mass * (radius*radius)}" />
-      </inertial>
-  </xacro:macro>
+<material name="black">
+    <color rgba="0.2 0.2 0.2 1.0"/>
+</material>
 <!-- ===================== MAIN BODY =========================== -->
   <link name="base_footprint"/>
@@ -45,5 +10,5 @@
     <parent link="base_footprint"/>
     <child link="base_link"/>
-    <origin xyz="0 0 0.041" rpy="0 0 0"/>
+    <origin xyz="0 0 0.042" rpy="0 0 0"/>
   </joint>
   <!-- CHASSIS -->
@@ -51,8 +16,7 @@
     <visual>
       <geometry>
-        <box size="0.18 0.13 0.095"/>
+        <mesh filename="package://mbot_description/meshes/mbot-classic-simplied.dae"/>
       </geometry>
-      <origin rpy="0 0 0" xyz="-0.045 0 0.0275"/>
-      <material name="blue"/>
+      <origin rpy="0 0 0" xyz="-0.04 -0.115 0.005"/>
     </visual>
     <collision>
@@ -60,46 +24,44 @@
         <box size="0.18 0.13 0.095"/>
       </geometry>
-      <origin rpy="0 0 0" xyz="-0.045 0 0.0275"/>
+      <origin rpy="0 0 0" xyz="-0.04 -0.115 0.005"/>
     </collision>
-    <xacro:inertial_box mass="0.3" x="0.18" y="0.13" z="0.095">
-      <origin xyz="0 0 0.0275" rpy="0 0 0"/>
-    </xacro:inertial_box>
   </link>
+  <!-- CAMERA -->
+  <link name="camera_link"/>
+  <joint name="camera_joint" type="fixed">
+    <parent link="base_link"/>
+    <child link="camera_link"/>
+    <origin xyz="0.05751 0 0.02936" rpy="0 0 0"/>
+  </joint>
   <!-- WHEELS -->
   <link name="left_wheel_link">
     <visual>
       <geometry>
-        <cylinder radius="0.041" length="0.02"/>
+        <mesh filename="package://mbot_description/meshes/wheel_l.stl" scale="0.001 0.001 0.001"/>
       </geometry>
-      <origin rpy="0 0 0" xyz="0 0 0"/>
+      <origin rpy="0 0 0" xyz="0 0 0.0115"/>
       <material name="black"/>
     </visual>
     <collision>
       <geometry>
-        <cylinder radius="0.041" length="0.02"/>
+        <cylinder radius="0.042" length="0.024"/>
       </geometry>
-      <origin rpy="0 0 0" xyz="0 0 0"/>
+      <origin rpy="0 0 0" xyz="0 0 0.0115"/>
     </collision>
-    <xacro:inertial_cylinder mass="0.1" length="0.02" radius="0.041">
-      <origin xyz="0 0 0" rpy="0 0 0"/>
-    </xacro:inertial_cylinder>
-  </link>
+      </link>
   <link name="right_wheel_link">
     <visual>
       <geometry>
-        <cylinder radius="0.041" length="0.02"/>
+        <mesh filename="package://mbot_description/meshes/wheel_r.stl" scale="0.001 0.001 0.001"/>
       </geometry>
-      <origin rpy="0 0 0" xyz="0 0 0"/>
+      <origin rpy="0 0 0" xyz="0 0 0.0115"/>
       <material name="black"/>
     </visual>
     <collision>
       <geometry>
-        <cylinder radius="0.041" length="0.02"/>
+        <cylinder radius="0.042" length="0.024"/>
       </geometry>
-      <origin rpy="0 0 0" xyz="0 0 0"/>
+      <origin rpy="0 0 0" xyz="0 0 0.0115"/>
     </collision>
-    <xacro:inertial_cylinder mass="0.1" length="0.02" radius="0.041">
-      <origin xyz="0 0 0" rpy="0 0 0"/>
-    </xacro:inertial_cylinder>
   </link>
   <joint name="left_wheel_joint" type="continuous">
@@ -108,6 +70,4 @@
     <origin xyz="0 0.085 0" rpy="-1.5708 0 0"/>
     <axis xyz="0 0 1"/>
-    <limit effort="5000" velocity="10"/>
-    <dynamics damping="1.0" friction="1.0"/>
   </joint>
   <joint name="right_wheel_joint" type="continuous">
@@ -116,53 +76,11 @@
     <origin xyz="0 -0.085 0" rpy="1.5708 0 0"/>
     <axis xyz="0 0 -1"/>
-    <limit effort="5000" velocity="10"/>
-    <dynamics damping="1.0" friction="1.0"/>
   </joint>
-  <!-- CASTER (Support ball that can roll freely) -->
-  <!-- Set to fixed joint but also set friction to 0 -->
-  <joint name="caster_wheel_joint" type="fixed">
-    <parent link="base_link"/>
-    <child link="caster_wheel_link"/>
-    <origin xyz="-0.09 0 0"/>
-  </joint>
-  <link name="caster_wheel_link">
-    <visual>
-      <geometry>
-        <sphere radius="0.041"/>
-      </geometry>
-      <material name="black"/>
-    </visual>
-    <collision>
-      <geometry>
-        <sphere radius="0.041"/>
-      </geometry>
-    </collision>
-    <xacro:inertial_sphere mass="0.1" radius="0.041">
-      <origin xyz="0 0 0" rpy="0 0 0"/>
-    </xacro:inertial_sphere>
-  </link>
   <!-- RPLidar A1 (Directly above base_link) -->
-  <link name="lidar_link">
-    <visual>
-      <geometry>
-        <cylinder radius="0.049" length="0.041"/>
-      </geometry>
-      <origin rpy="0 0 0" xyz="0 0 0"/>
-      <material name="black"/>
-    </visual>
-    <collision>
-      <geometry>
-        <cylinder radius="0.049" length="0.041"/>
-      </geometry>
-      <origin rpy="0 0 0" xyz="0 0 0"/>
-    </collision>
-    <xacro:inertial_cylinder mass="0.1" length="0.041" radius="0.049">
-      <origin xyz="0 0 0" rpy="0 0 0"/>
-    </xacro:inertial_cylinder>
-  </link>
+  <link name="lidar_link"/>
   <joint name="lidar_joint" type="fixed">
     <parent link="base_link"/>
     <child link="lidar_link"/>
-    <origin xyz="0 0 0.1" rpy="0 0 3.14"/>
+    <origin xyz="0 0 0.14179" rpy="0 0 3.14"/>
   </joint>
 </robot>

Commit message: add apriltag detection

File: mbot_description/urdf/mbot_classic.urdf.xacro (robot description, xacro)
@@ -28,9 +28,9 @@
   </link>
   <!-- CAMERA -->
-  <link name="camera_link"/>
+  <link name="camera"/>
   <joint name="camera_joint" type="fixed">
     <parent link="base_link"/>
-    <child link="camera_link"/>
-    <origin xyz="0.05751 0 0.02936" rpy="0 0 0"/>
+    <child link="camera"/>
+    <origin xyz="0.05751 0 0.02936" rpy="3.14 -1.57 0"/>
   </joint>
   <!-- WHEELS -->

Commit message: correct the camera transform

File: mbot_description/urdf/mbot_classic.urdf.xacro (robot description, xacro)
@@ -32,5 +32,5 @@
     <parent link="base_link"/>
     <child link="camera"/>
-    <origin xyz="0.05751 0 0.02936" rpy="3.14 -1.57 0"/>
+    <origin xyz="0.05751 0 0.02936" rpy="-1.57 0 -1.57"/>
   </joint>
   <!-- WHEELS -->
