Commit message: Added camera driver + apriltag (#6)
* Add camera_ros as a submodule

* add apriltag detection

* correct the camera transform

File: mbot_description/urdf/mbot_classic.urdf.xacro (robot description, xacro)
@@ -28,9 +28,9 @@
   </link>
   <!-- CAMERA -->
-  <link name="camera_link"/>
+  <link name="camera"/>
   <joint name="camera_joint" type="fixed">
     <parent link="base_link"/>
-    <child link="camera_link"/>
-    <origin xyz="0.05751 0 0.02936" rpy="0 0 0"/>
+    <child link="camera"/>
+    <origin xyz="0.05751 0 0.02936" rpy="-1.57 0 -1.57"/>
   </joint>
   <!-- WHEELS -->
